Commit message: surrendered to ignition, integrating python_api

File: src/barrier_control/urdf/my_robot.urdf.xacro (robot description, xacro)
@@ -1,79 +1,158 @@
-<?xml version="1.0"?>
-<robot xmlns:xacro="http://www.ros.org/wiki/xacro" name="my_robot">
-  <link name="base_link">
+<?xml version="1.0" ?>
+<robot name="cartopole">
+  <link name="slideBar">
     <visual>
       <geometry>
-        <box size="0.5 0.3 0.2"/>
+        <box size="30 0.05 0.05"/>
       </geometry>
-      <material name="blue">
-        <color rgba="0.1 0.1 0.8 1"/>
-      </material>
+      <origin xyz="0 0 1"/>
+    </visual>
+    <inertial>
+      <mass value="100"/>
+      <inertia ixx="1.0" ixy="0.0" ixz="0.0" iyy="1.0" iyz="0.0" izz="1.0"/>
+    </inertial>
+  </link>
+  <link name="cart">
+    <visual>
+      <geometry>
+        <box size="0.5 0.5 0.2"/>
+      </geometry>
+      <origin xyz="0 0 1"/>
+    </visual>
+    <inertial>
+      <mass value="1"/>
+      <inertia ixx="1.0" ixy="0.0" ixz="0.0" iyy="1.0" iyz="0.0" izz="1.0"/>
+    </inertial>
+  </link>
+  <link name="leg1">
+    <visual>
+      <geometry>
+        <cylinder radius="0.2" length="1.0"/>
+      </geometry>
+      <origin xyz="0 0 0"/>
     </visual>
     <collision>
       <geometry>
-        <box size="0.5 0.3 0.2"/>
+        <cylinder radius="0.2" length="1.0"/>
       </geometry>
+      <origin xyz="0 0 0"/>
     </collision>
     <inertial>
-      <mass value="1.0"/>
-      <inertia ixx="0.01" ixy="0.0" ixz="0.0" iyy="0.01" iyz="0.0" izz="0.01"/>
+      <mass value="1"/>
+      <inertia ixx="1.0" ixy="0.0" ixz="0.0" iyy="1.0" iyz="0.0" izz="1.0"/>
     </inertial>
   </link>
-  <xacro:macro name="wheel_link" params="prefix reflect_x">
-    <link name="${prefix}_wheel_link">
-      <visual>
-        <origin xyz="0 0 0" rpy="${pi/2} 0 0"/>
-        <geometry>
-          <cylinder radius="0.1" length="0.05"/>
-        </geometry>
-        <material name="black">
-          <color rgba="0.1 0.1 0.1 1"/>
-        </material>
-      </visual>
-      <collision>
-        <origin xyz="0 0 0" rpy="${pi/2} 0 0"/>
-        <geometry>
-          <cylinder radius="0.1" length="0.05"/>
-        </geometry>
-      </collision>
-      <inertial>
-        <mass value="0.2"/>
-        <inertia ixx="0.001" ixy="0.0" ixz="0.0" iyy="0.001" iyz="0.0" izz="0.002"/>
-      </inertial>
-    </link>
-  </xacro:macro>
-  <xacro:wheel_link prefix="front_left" reflect_x="1"/>
-  <xacro:wheel_link prefix="front_right" reflect_x="-1"/>
-  <joint name="base_to_front_left_wheel" type="continuous">
-    <parent link="base_link"/>
-    <child link="front_left_wheel_link"/>
-    <origin xyz="0.2 ${0.15 + 0.025} -0.05" rpy="0 0 0"/> <axis xyz="0 1 0"/>
+  <link name="leg2">
+    <visual>
+      <geometry>
+        <cylinder radius="0.2" length="1.0"/>
+      </geometry>
+      <origin xyz="0 0 0"/>
+    </visual>
+    <collision>
+      <geometry>
+        <cylinder radius="0.2" length="1.0"/>
+      </geometry>
+      <origin xyz="0 0 0"/>
+    </collision>
+    <inertial>
+      <mass value="1"/>
+      <inertia ixx="1.0" ixy="0.0" ixz="0.0" iyy="1.0" iyz="0.0" izz="1.0"/>
+    </inertial>
+  </link>
+  <joint name="slider_to_cart" type="prismatic">
+    <axis xyz="1 0 0"/>
+    <origin xyz="0.0 0.0 0.0"/>
+    <parent link="slideBar"/>
+    <child link="cart"/>
+    <limit effort="1000.0" lower="-15" upper="15" velocity="30"/>
+    <dynamics damping="0.0" friction="0.0"/>
   </joint>
-  <joint name="base_to_front_right_wheel" type="continuous">
-    <parent link="base_link"/>
-    <child link="front_right_wheel_link"/>
-    <origin xyz="0.2 ${-(0.15 + 0.025)} -0.05" rpy="0 0 0"/>
-    <axis xyz="0 1 0"/>
+  <link name="imu">
+    <inertial>
+      <mass value="0.1"/>
+      <inertia ixx="1.0" ixy="0" ixz="0" iyy="1.0" iyz="0" izz="1.0"/>
+    </inertial>
+  </link>
+  <joint name="cart_to_imu" type="fixed">
+    <origin xyz="0.0 0.0 0.0"/>
+    <parent link="cart"/>
+    <child link="imu"/>
+    <dynamics damping="0.0" friction="0.0"/>
   </joint>
+  <joint name="slider_to_leg1" type="fixed">
+    <origin xyz="-15.0 0.0 0.5"/>
+    <parent link="slideBar"/>
+    <child link="leg1"/>
+    <dynamics damping="0.0" friction="0.0"/>
+  </joint>
+  <joint name="slider_to_leg2" type="fixed">
+    <origin xyz="15 0.0 0.5"/>
+    <parent link="slideBar"/>
+    <child link="leg2"/>
+    <dynamics damping="0.0" friction="0.0"/>
+  </joint>
+  <gazebo reference="imu">
+    <sensor name="cart_imu_sensor" type="imu">
+      <always_on>1</always_on>
+      <update_rate>10.0</update_rate>
+      <visualize>true</visualize>
+      <topic>imu</topic>
+    </sensor>
+  </gazebo>
+  <ros2_control name="GazeboSimSystem" type="system">
+    <hardware>
+      <plugin>gz_ros2_control/GazeboSimSystem</plugin>
+    </hardware>
+    <joint name="slider_to_cart">
+      <command_interface name="velocity">
+        <param name="min">-15</param>
+        <param name="max">15</param>
+      </command_interface>
+      <state_interface name="position">
+        <param name="initial_value">1.0</param>
+      </state_interface>
+      <state_interface name="velocity"/>
+      <state_interface name="effort"/>
+    </joint>
+    <sensor name="cart_imu_sensor">
+      <state_interface name="orientation.x"/>
+      <state_interface name="orientation.y"/>
+      <state_interface name="orientation.z"/>
+      <state_interface name="orientation.w"/>
+      <state_interface name="angular_velocity.x"/>
+      <state_interface name="angular_velocity.y"/>
+      <state_interface name="angular_velocity.z"/>
+      <state_interface name="linear_acceleration.x"/>
+      <state_interface name="linear_acceleration.y"/>
+      <state_interface name="linear_acceleration.z"/>
+    </sensor>
+  </ros2_control>
+  <gazebo reference="slideBar">
+    <visual>
+      <material>
+        <ambient>0 0.8 0 1</ambient>
+        <diffuse>0 0.8 0 1</diffuse>
+        <specular>0 0.8 0 1</specular>
+      </material>
+    </visual>
+  </gazebo>
+  <gazebo reference="cart">
+    <visual>
+      <material>
+        <ambient>0 0 0.8 1</ambient>
+        <diffuse>0 0 0.8 1</diffuse>
+        <specular>0 0 0.8 1</specular>
+      </material>
+    </visual>
+  </gazebo>
   <gazebo>
-    <plugin filename="libgazebo_ros2_control.so" name="gazebo_ros2_control">
-      <robot_param>robot_description</robot_param>
-      <robot_param_node>robot_state_publisher</robot_param_node>
-      </plugin>
-  </gazebo>
-  <gazebo reference="base_link">
-    <material>Gazebo/Blue</material>
-    <mu1>0.2</mu1>
-    <mu2>0.2</mu2>
-  </gazebo>
-  <gazebo reference="front_left_wheel_link">
-    <material>Gazebo/Black</material>
-    <mu1>1.0</mu1>
-    <mu2>1.0</mu2>
-  </gazebo>
-   <gazebo reference="front_right_wheel_link">
-    <material>Gazebo/Black</material>
-    <mu1>1.0</mu1>
-    <mu2>1.0</mu2>
+    <plugin filename="gz_ros2_control-system" name="gz_ros2_control::GazeboSimROS2ControlPlugin">
+      <parameters>$(find barrier_control)/config/cart_controller_velocity.yaml</parameters>
+    </plugin>
+    <plugin
+      filename="ignition-gazebo-imu-system"
+      name="ignition::gazebo::systems::Imu">
+    </plugin>
   </gazebo>
 </robot>

File: src/kortex_description/arms/gen3/6dof/urdf/gen3_macro.xacro (robot description, xacro)
@@ -30,5 +30,6 @@
     use_external_cable:=false
     initial_positions:=${dict(joint_1=0.0,joint_2=0.0,joint_3=0.0,joint_4=0.0,joint_5=0.0,joint_6=0.0)}
-    moveit_active:=false">
+    moveit_active:=false
+    robot_controller:=robot1_controllers.yaml">
     <!-- ros2 control include -->
     <xacro:include filename="$(find kortex_description)/arms/gen3/${dof}dof/urdf/kortex.ros2_control.xacro" />
@@ -54,5 +55,7 @@
       gripper_max_velocity="${gripper_max_velocity}"
       gripper_max_force="${gripper_max_force}"
-      gripper_joint_name="${gripper_joint_name}"/>
+      gripper_joint_name="${gripper_joint_name}"
+      robot_controller="${robot_controller}"
+      />
     <joint name="${prefix}base_joint" type="fixed">
       <xacro:insert_block name="origin" />

File: src/kortex_description/arms/gen3/6dof/urdf/kortex.ros2_control.xacro (robot description, xacro)
@@ -24,9 +24,11 @@
     gripper_max_velocity:=100.0
     gripper_max_force:=100.0
-    moveit_active:=false">
+    moveit_active:=false
+    robot_controller:=robot1_controllers.yaml"
+    >
     <ros2_control name="${name}" type="system">
       <hardware>
         <xacro:if value="${sim_ignition}">
-          <plugin>ign_ros2_control/IgnitionSystem</plugin>
+          <plugin>gz_ros2_control/GazeboSimSystem</plugin>
         </xacro:if>
         <xacro:if value="${sim_gazebo}">
@@ -182,4 +184,9 @@
       </xacro:if>
     </ros2_control>
+    <gazebo>
+      <plugin filename="gz_ros2_control-system" name="gz_ros2_control::GazeboSimROS2ControlPlugin">
+        <parameters>$(find ros_gz_sim_demos)/config/${robot_controller}</parameters>
+      </plugin>
+    </gazebo>
   </xacro:macro>
 </robot>

File: src/kortex_description/robots/gen3.xacro (robot description, xacro)
@@ -24,4 +24,5 @@
     <xacro:arg name="use_internal_bus_gripper_comm" default="false" />
     <xacro:arg name="use_external_cable" default="false" />
+    <xacro:arg name="robot_controller" default="robot1_controllers.yaml" />
     <!-- Arguments for initial pose of the robot relative to its parent link (world) -->
     <xacro:arg name="initial_pose_x" default="0.0"/>
@@ -61,5 +62,6 @@
         sim_isaac="$(arg sim_isaac)"
         use_external_cable="$(arg use_external_cable)"
-        initial_positions="${xacro.load_yaml(initial_positions_file)}">
+        initial_positions="${xacro.load_yaml(initial_positions_file)}"
+        robot_controller="$(arg robot_controller)">
         <origin xyz="$(arg initial_pose_x) $(arg initial_pose_y) $(arg initial_pose_z)"
                 rpy="$(arg initial_pose_roll) $(arg initial_pose_pitch) $(arg initial_pose_yaw)" />

File: src/kortex_description/robots/kinova.urdf.xacro (robot description, xacro)
@@ -76,5 +76,5 @@
     </gazebo>
   </xacro:if>
-  <xacro:if value="$(arg sim_ignition)">
+  <!-- <xacro:if value="$(arg sim_ignition)">
     <!-- Gazebo plugins -->
     <gazebo reference="world">
@@ -150,4 +150,4 @@
       </sensor>
     </gazebo>
-  </xacro:if>
+  </xacro:if> -->
 </robot>

File: src/kortex_description/robots/kortex_robot.xacro (robot description, xacro)
@@ -30,5 +30,6 @@
     gripper_max_force:=100.0
     gripper_com_port:=/dev/ttyUSB0
-    moveit_active:=false">
+    moveit_active:=false
+    robot_controller:=robot1_controllers.yaml">
     <!-- Include and load arm macro files -->
     <xacro:include filename="$(find kortex_description)/arms/${arm}/${dof}dof/urdf/${arm}_macro.xacro" />
@@ -59,5 +60,6 @@
       use_external_cable="${use_external_cable}"
       initial_positions="${initial_positions}"
-      moveit_active="${moveit_active}">
+      moveit_active="${moveit_active}"
+      robot_controller="${robot_controller}">
       <xacro:insert_block name="origin" />
     </xacro:load_arm>
