Commit message: Transition to trajectory_controller

File: src/kortex_description/arms/gen3/6dof/urdf/gen3_macro.xacro (robot description, xacro)
@@ -344,5 +344,5 @@
       </joint>
     </xacro:unless>
-    <link name="${prefix}end_effector_link" />
+    <link name="${prefix}end_effector_link"/>
     <joint
       name="${prefix}end_effector"

File: src/kortex_description/arms/gen3/6dof/urdf/kortex.ros2_control.xacro (robot description, xacro)
@@ -67,110 +67,104 @@
       </hardware>
       <joint name="${prefix}joint_1">
+        <command_interface name="position">
+          <param name="min">{-2*pi}</param>
+          <param name="max">{2*pi}</param>
+        </command_interface>
         <command_interface name="velocity">
           <param name="min">-0.8727</param>  <!-- Adjust limits as needed -->
           <param name="max">0.8727</param>
         </command_interface>
-        <xacro:if value="${sim_gazebo or use_fake_hardware}">
-          <state_interface name="position">
-            <param name="initial_value">${initial_positions['joint_1']}</param>
-          </state_interface>
-          <state_interface name="velocity">
-            <param name="initial_value">0.0</param>  <!-- Add this line -->
-          </state_interface>
-        </xacro:if>
-        <xacro:unless value="${sim_gazebo or use_fake_hardware}">
-          <state_interface name="position"/>
-          <state_interface name="velocity"/>
-        </xacro:unless>
+        <state_interface name="position">
+          <param name="initial_value">${initial_positions['joint_1']}</param>
+        </state_interface>
+        <state_interface name="velocity">
+          <param name="initial_value">0.0</param>
+        </state_interface>
+        <state_interface name="effort"/>
       </joint>
       <joint name="${prefix}joint_2">
+        <command_interface name="position">
+          <param name="min">-2.41</param>
+          <param name="max">2.41</param>
+        </command_interface>
         <command_interface name="velocity">
           <param name="min">-0.8727</param>  <!-- Adjust limits as needed -->
           <param name="max">0.8727</param>
         </command_interface>
-        <xacro:if value="${sim_gazebo or use_fake_hardware}">
-          <state_interface name="position">
-            <param name="initial_value">${initial_positions['joint_2']}</param>
-          </state_interface>
-          <state_interface name="velocity">
-            <param name="initial_value">0.0</param>  <!-- Add this line -->
-          </state_interface>
-        </xacro:if>
-        <xacro:unless value="${sim_gazebo or use_fake_hardware}">
-          <state_interface name="position"/>
-          <state_interface name="velocity"/>
-        </xacro:unless>
+        <state_interface name="position">
+          <param name="initial_value">${initial_positions['joint_2']}</param>
+        </state_interface>
+        <state_interface name="velocity">
+          <param name="initial_value">0.0</param>  <!-- Add this line -->
+        </state_interface>
+        <state_interface name="effort"/>
       </joint>
       <joint name="${prefix}joint_3">
+        <command_interface name="position">
+          <param name="min">-2.66</param>
+          <param name="max">2.66</param>
+        </command_interface>
         <command_interface name="velocity">
           <param name="min">-0.8727</param>  <!-- Adjust limits as needed -->
           <param name="max">0.8727</param>
         </command_interface>
-        <xacro:if value="${sim_gazebo or use_fake_hardware}">
-          <state_interface name="position">
-            <param name="initial_value">${initial_positions['joint_3']}</param>
-          </state_interface>
-          <state_interface name="velocity">
-            <param name="initial_value">0.0</param>  <!-- Add this line -->
-          </state_interface>
-        </xacro:if>
-        <xacro:unless value="${sim_gazebo or use_fake_hardware}">
-          <state_interface name="position"/>
-          <state_interface name="velocity"/>
-        </xacro:unless>
+        <state_interface name="position">
+          <param name="initial_value">${initial_positions['joint_3']}</param>
+        </state_interface>
+        <state_interface name="velocity">
+          <param name="initial_value">0.0</param>  <!-- Add this line -->
+        </state_interface>
+        <state_interface name="effort"/>
       </joint>
       <joint name="${prefix}joint_4">
+        <command_interface name="position">
+          <param name="min">{-2*pi}</param>
+          <param name="max">{2*pi}</param>
+        </command_interface>
         <command_interface name="velocity">
           <param name="min">-0.8727</param>  <!-- Adjust limits as needed -->
           <param name="max">0.8727</param>
         </command_interface>
-        <xacro:if value="${sim_gazebo or use_fake_hardware}">
-          <state_interface name="position">
-            <param name="initial_value">${initial_positions['joint_4']}</param>
-          </state_interface>
-          <state_interface name="velocity">
-            <param name="initial_value">0.0</param>  <!-- Add this line -->
-          </state_interface>
-        </xacro:if>
-        <xacro:unless value="${sim_gazebo or use_fake_hardware}">
-          <state_interface name="position"/>
-          <state_interface name="velocity"/>
-        </xacro:unless>
+        <state_interface name="position">
+          <param name="initial_value">${initial_positions['joint_4']}</param>
+        </state_interface>
+        <state_interface name="velocity">
+          <param name="initial_value">0.0</param>  <!-- Add this line -->
+        </state_interface>
+        <state_interface name="effort"/>
       </joint>
       <joint name="${prefix}joint_5">
+        <command_interface name="position">
+          <param name="min">-2.23</param>
+          <param name="max">2.23</param>
+        </command_interface>
         <command_interface name="velocity">
           <param name="min">-0.8727</param>  <!-- Adjust limits as needed -->
           <param name="max">0.8727</param>
         </command_interface>
-        <xacro:if value="${sim_gazebo or use_fake_hardware}">
-          <state_interface name="position">
-            <param name="initial_value">${initial_positions['joint_5']}</param>
-          </state_interface>
-          <state_interface name="velocity">
-            <param name="initial_value">0.0</param>  <!-- Add this line -->
-          </state_interface>
-        </xacro:if>
-        <xacro:unless value="${sim_gazebo or use_fake_hardware}">
-          <state_interface name="position"/>
-          <state_interface name="velocity"/>
-        </xacro:unless>
+        <state_interface name="position">
+          <param name="initial_value">${initial_positions['joint_5']}</param>
+        </state_interface>
+        <state_interface name="velocity">
+          <param name="initial_value">0.0</param>  <!-- Add this line -->
+        </state_interface>
+        <state_interface name="effort"/>
       </joint>
       <joint name="${prefix}joint_6">
+        <command_interface name="position">
+          <param name="min">{-2*pi}</param>
+          <param name="max">{2*pi}</param>
+        </command_interface>
         <command_interface name="velocity">
           <param name="min">-0.8727</param>  <!-- Adjust limits as needed -->
           <param name="max">0.8727</param>
         </command_interface>
-        <xacro:if value="${sim_gazebo or use_fake_hardware}">
-          <state_interface name="position">
-            <param name="initial_value">${initial_positions['joint_6']}</param>
-          </state_interface>
-          <state_interface name="velocity">
-            <param name="initial_value">0.0</param>  <!-- Add this line -->
-          </state_interface>
-        </xacro:if>
-        <xacro:unless value="${sim_gazebo or use_fake_hardware}">
-          <state_interface name="position"/>
-          <state_interface name="velocity"/>
-        </xacro:unless>
+        <state_interface name="position">
+          <param name="initial_value">${initial_positions['joint_6']}</param>
+        </state_interface>
+        <state_interface name="velocity">
+          <param name="initial_value">0.0</param>  <!-- Add this line -->
+        </state_interface>
+        <state_interface name="effort"/>
       </joint>
       <xacro:if value="${use_internal_bus_gripper_comm}">

File: src/kortex_description/robots/gen3.xacro (robot description, xacro)
@@ -37,5 +37,5 @@
     <!-- convert to property to use substitution in function -->
     <xacro:property name="initial_positions_file" default="$(arg initial_positions_file)"/>
-    <link name="world" />
+    <link name="world"/>
     <xacro:load_robot
         parent="world"

File: src/kortex_description/robots/kinova.urdf.xacro (robot description, xacro)
@@ -38,5 +38,5 @@
   <xacro:property name="initial_positions_file" default="$(arg initial_positions_file)"/>
   <!-- create link fixed to the "world" -->
-  <link name="world" />
+  <link name="world"/>
   <xacro:load_robot
     parent="world"
